File: Circuit Design/PCBDesign/LFRCircuit/LFRCircuit.kicad_sch (KiCad schematic)
At the start: 32 parts, among them J1 OLED_128x64, M1 Motor_DC, M2 Motor_DC, U1 L293D, U2 TPS54202DDC

Commit message: Tweaked a little bit
Connections:
- net 12Vout is gone; now on net +12V: INA1.2 (IN-), INA1.3 (VBS)
- net +12V: no longer BT3.1 (+), INA1.1 (IN+)
- new net BatOUT: BT3.1 (+), INA1.1 (IN+)
Changed lines of the file:
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@@
 		)
 	)
-	(label "12Vout"
+	(label "+12V"
 		(at 80.01 39.37 0)
 		(effects
@@
 		(on_board yes)
 		(dnp no)
-		(fields_autoplaced yes)
 		(property "Reference" "#PWR026"
 			(at 88.9 96.52 0)
@@
 			)
 		)
-		(property "Value" "+12V"
-			(at 88.9 87.63 0)
-			(effects
-				(font
-					(size 1.27 1.27)
-				)
+		(property "Value" "BatOUT"
+			(at 85.598 88.392 0)
+			(effects
+				(font
+					(size 1.27 1.27)
+				)
+				(justify left)
 			)
 		)
@@
 		(on_board yes)
 		(dnp no)
-		(fields_autoplaced yes)
 		(property "Reference" "#PWR07"
 			(at 91.44 34.29 0)
@@
 			)
 		)
-		(property "Value" "+12V"
-			(at 83.82 34.2899 90)
-			(effects
-				(font
-					(size 1.27 1.27)
-				)
-				(justify left)
-			)
-		)
+		(property "Value" "BatOUT"
+			(at 81.026 34.036 90)
+			(effects
+				(font
+					(size 1.27 1.27)
+				)
+			)
+		)

Commit message: Updated PCB
Parts:
- removed C3: 10uF, Capacitor_SMD:C_1206_3216Metric_Pad1.33x1.80mm_HandSolder, symbol Device:C
- removed C4, C5: 0.1uF, Capacitor_SMD:C_1206_3216Metric_Pad1.33x1.80mm_HandSolder, symbol Device:C
- removed C6, C7: 22uF, Capacitor_SMD:C_1206_3216Metric_Pad1.33x1.80mm_HandSolder, symbol Device:C
- removed C8: 75pF, Capacitor_SMD:C_1206_3216Metric_Pad1.33x1.80mm_HandSolder, symbol Device:C
- removed D5: D, Diode_SMD:D_1206_3216Metric_Pad1.42x1.75mm_HandSolder, symbol Device:D
- removed L1: 15uH, Inductor_SMD:L_1206_3216Metric_Pad1.42x1.75mm_HandSolder, symbol Device:L
- removed R1: 49.9, Resistor_SMD:R_1206_3216Metric_Pad1.30x1.75mm_HandSolder, symbol Device:R
- removed R2: 100K, Resistor_SMD:R_1206_3216Metric_Pad1.30x1.75mm_HandSolder, symbol Device:R
- removed R3: 13.3K, Resistor_SMD:R_1206_3216Metric_Pad1.30x1.75mm_HandSolder, symbol Device:R
- removed R4: 511K, Resistor_SMD:R_1206_3216Metric_Pad1.30x1.75mm_HandSolder, symbol Device:R
- removed R5: 105K, Resistor_SMD:R_1206_3216Metric_Pad1.30x1.75mm_HandSolder, symbol Device:R
- removed U2: TPS54202DDC, Package_TO_SOT_SMD:SOT-23-6, symbol Regulator_Switching:TPS54202DDC
- added U2: ~, Connector_JST:JST_XH_B3B-XH-A_1x03_P2.50mm_Vertical, symbol PowerConverter:buckConverter
- ArduinoNanoTypeC1: footprint ArduinoNano:ArduinoNanoTypeC -> RactangularPad:ArduinoNanoRactangularPads
- BT1, BT2, BT3: footprint Connector_JST:JST_XH_S2B-XH-A_1x02_P2.50mm_Horizontal -> RactangularPad:JST_XH_B2B-XH-A_1x02_P2.50mm_Vertical_ractangular
- C1, C2: footprint Capacitor_SMD:C_1206_3216Metric_Pad1.33x1.80mm_HandSolder -> Capacitor_THT:C_Disc_D5.0mm_W2.5mm_P5.00mm
- D1, D2, D3, D4: footprint Diode_SMD:D_1206_3216Metric_Pad1.42x1.75mm_HandSolder -> Diode_THT:D_DO-41_SOD81_P7.62mm_Horizontal
- INA1: footprint Connector_PinSocket_2.54mm:PinSocket_1x08_P2.54mm_Vertical -> RactangularPad:PinSocket_1x08_P2.54mm_Vertical_ractangular
- IRSensor6Array1: footprint Connector_JST:JST_XH_S8B-XH-A_1x08_P2.50mm_Horizontal -> Connector_JST:JST_XH_B8B-XH-A_1x08_P2.50mm_Vertical
- M1, M2: footprint Connector_JST:JST_XH_S2B-XH-A-1_1x02_P2.50mm_Horizontal -> RactangularPad:JST_XH_B2B-XH-A_1x02_P2.50mm_Vertical_ractangular
- RotaryEncoder1: footprint Connector_JST:JST_XH_S5B-XH-A-1_1x05_P2.50mm_Horizontal -> Connector_JST:JST_XH_B5B-XH-A_1x05_P2.50mm_Vertical
- SonarSensor3Array1: footprint Connector_JST:JST_XH_S5B-XH-A_1x05_P2.50mm_Horizontal -> Connector_JST:JST_XH_B5B-XH-A_1x05_P2.50mm_Vertical
- U1: footprint Package_DIP:DIP-16_W7.62mm -> RactangularPad:DIP-16_W7.62mm_ractangularPads
Connections:
- net +12V: now also U2.1 (IN+)
- net +5V: now also U2.3 (OUT+)
- net GND: now also U2.2 (IN-); no longer ArduinoNanoTypeC1.29 (GND )
- no-connect marks 8 -> 9
